Commit message: Reading enabled, writing needs rework

File: description/ros2_control/r6bot.ros2_control.xacro (robot description, xacro)
@@ -8,6 +8,6 @@
       <joint name="joint_1">
         <command_interface name="position">
-          <!-- <param name="min">${-2*pi}</param>
-          <param name="max">${2*pi}</param> -->
+          <param name="min">${-pi}</param>
+          <param name="max">${pi}</param>
         </command_interface>
         <command_interface name="velocity">
@@ -22,6 +22,6 @@
       <joint name="joint_2">
         <command_interface name="position">
-          <!-- <param name="min">${-2*pi}</param>
-          <param name="max">${2*pi}</param> -->
+          <param name="min">-1.13446</param>
+          <param name="max">1.22173</param>
         </command_interface>
         <command_interface name="velocity">
@@ -36,6 +36,6 @@
       <joint name="joint_3">
         <command_interface name="position">
-          <!-- <param name="min">${-pi}</param>
-          <param name="max">${pi}</param> -->
+          <param name="min">-2.07694</param>
+          <param name="max">1.578</param>
         </command_interface>
         <command_interface name="velocity">
@@ -50,6 +50,6 @@
       <joint name="joint_4">
         <command_interface name="position">
-          <!-- <param name="min">${-2*pi}</param>
-          <param name="max">${2*pi}</param> -->
+          <param name="min">-4.88692</param>
+          <param name="max">4.88692</param>
         </command_interface>
         <command_interface name="velocity">
@@ -64,6 +64,6 @@
       <joint name="joint_5">
         <command_interface name="position">
-          <!-- <param name="min">${-2*pi}</param>
-          <param name="max">${2*pi}</param> -->
+          <param name="min">-2.18166</param>
+          <param name="max">2.18166</param>
         </command_interface>
         <command_interface name="velocity">
@@ -78,6 +78,6 @@
       <joint name="joint_6">
         <command_interface name="position">
-          <!-- <param name="min">${-2*pi}</param>
-          <param name="max">${2*pi}</param> -->
+          <param name="min">${-2*pi}</param>
+          <param name="max">${2*pi}</param>
         </command_interface>
         <command_interface name="velocity">

File: description/urdf/khi_ux150_description.urdf.xacro (robot description, xacro)
@@ -176,5 +176,5 @@
       <child link="link_2"/>
       <axis xyz="0.0 1.0 0.0"/>
-      <limit lower="-1.22173" upper="1.13446" effort="1000" velocity="1"/>
+      <limit lower="-1.13446" upper="1.22173" effort="1000" velocity="1"/>
   </joint>
   <!-- <joint name="joint_2_2" type="revolute">
@@ -183,5 +183,4 @@
       <child link="${prefix}parallel_2"/>
       <axis xyz="0.0 -1.0 0.0"/>
-      <limit lower="-1.22173" upper="1.13446" effort="1000" velocity="1"/>
       <mimic joint="jointt2" multiplier="1.0"/>
   </joint> -->
@@ -191,5 +190,5 @@
       <child link="link_3"/>
       <axis xyz="0.0 -1.0 0.0"/>
-      <limit lower="-1.22173" upper="1.13446" effort="1000" velocity="1"/>
+      <limit lower="-1.13446" upper="1.22173" effort="1000" velocity="1"/>
       <mimic joint="joint_2" multiplier="1.0"/>
   </joint>
@@ -199,5 +198,5 @@
       <child link="link_4"/>
       <axis xyz="0.0 -1.0 0.0"/>
-      <limit lower="-1.578" upper="2.07694" effort="1000" velocity="1"/>
+      <limit lower="-2.07694" upper="1.578" effort="1000" velocity="1"/>
   </joint>
   <joint name="joint_4" type="revolute">
